File: hardware/dcpu.sch (KiCad schematic (older format))
At the start: 0 parts

Commit message: Hmm, seem to have changed the schematics again but not a clue what I did...
Changed lines of the file:
@@
-EESchema Schematic File Version 2  date Fri 19 Oct 2012 23:31:17 BST
+EESchema Schematic File Version 2  date Sun 31 Mar 2013 02:03:27 BST
 LIBS:power
 LIBS:device
@@
 LIBS:BS62LV256
 LIBS:dcpu-cache
-EELAYER 25  0
+EELAYER 27 0
 EELAYER END
-$Descr A4 11700 8267
+$Descr A4 11693 8268
 encoding utf-8
 Sheet 1 16
 Title "DCPU"
-Date "19 oct 2012"
+Date "30 mar 2013"
 Rev "A"
 Comp "David Robertson"
@@
 F 0 "#PWR01" H 3400 7250 30  0001 C CNN
 F 1 "GND" H 3400 7180 30  0001 C CNN
+F 2 "" H 3400 7250 60  0001 C CNN
+F 3 "" H 3400 7250 60  0001 C CNN
 	1    3400 7250
 	1    0    0    -1
@@
 F1 "REG-M.sch" 60
 F2 "LOAD-2" I L 3850 5400 60
-F3 "D7" I L 3850 4150 60
-F4 "D6" I L 3850 4050 60
-F5 "D5" I L 3850 3950 60
-F6 "D4" I L 3850 3850 60
-F7 "D3" I L 3850 3750 60
-F8 "D2" I L 3850 3650 60
-F9 "D1" I L 3850 3550 60
-F10 "D0" I L 3850 3450 60
+F3 "D7" B L 3850 4150 60
+F4 "D6" B L 3850 4050 60
+F5 "D5" B L 3850 3950 60
+F6 "D4" B L 3850 3850 60
+F7 "D3" B L 3850 3750 60
+F8 "D2" B L 3850 3650 60
+F9 "D1" B L 3850 3550 60
+F10 "D0" B L 3850 3450 60
 F11 "LOAD-1" I L 3850 5300 60
 F12 "A0" O R 4850 3450 60
@@
 F 0 "#02" H 10950 6770 30  0001 C CNN
 F 1 "PWR_FLAG" H 10950 6730 30  0000 C CNN
+F 2 "" H 10950 6500 60  0001 C CNN
+F 3 "" H 10950 6500 60  0001 C CNN
 	1    10950 6500
 	1    0    0    -1
@@
 F 0 "#GND03" H 10950 6820 30  0001 C CNN
 F 1 "PWR_FLAG" H 10950 6780 30  0000 C CNN
+F 2 "" H 10950 6550 60  0001 C CNN
+F 3 "" H 10950 6550 60  0001 C CNN
 	1    10950 6550
 	-1   0    0    1
@@
 F 0 "#PWR04" H 10750 6650 30  0001 C CNN
 F 1 "GND" H 10750 6580 30  0001 C CNN
+F 2 "" H 10750 6650 60  0001 C CNN
+F 3 "" H 10750 6650 60  0001 C CNN
 	1    10750 6650
 	1    0    0    -1
@@
 F 0 "#PWR05" H 10750 6490 20  0001 C CNN
 F 1 "+5V" H 10750 6490 30  0000 C CNN
+F 2 "" H 10750 6400 60  0001 C CNN
+F 3 "" H 10750 6400 60  0001 C CNN
 	1    10750 6400
 	1    0    0    -1
